File: extras/kicad/Drv7Seg2x595.kicad_pcb (KiCad board)
At the start: 2 copper layers, 67.3 x 50.8 mm, 33 parts, among them IC1 74HC595, IC2 74HC595, Q1 MMBT3904, Q2 MMBT3904, Q3 MMBT3904, Q4 MMBT3904

Commit message: 1) Fix headers' and ICs' warnings on difference between ad hoc footprints and library, 2) Fix copper zones, 3) Add more informative header pins' text to silkscreen.
Other:
- board text added: "INTERFACE"
- board text added: "PWR_LED_JMP"
- board text removed: "PWRJMP"
