File: extras/kicad/Drv7Seg2x595.kicad_sch (KiCad schematic)
At the start: 33 parts, among them IC1 74HC595, IC2 74HC595, Q1 MMBT3904, Q2 MMBT3904, Q3 MMBT3904, Q4 MMBT3904

Commit message: Update BJT base resistors' value.
Parts:
- RT1, RT2, RT3, RT4: value 150 -> 1k5
Changed lines of the file:
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@@
 	(paper "A4")
 	(title_block
-		(date "01.12.2025")
+		(date "15.12.2025")
 		(comment 1 "Documentation: github.com/ErlingSigurdson/Drv7Seg2x595")
 		(comment 2 "Licensed under CERN-OHL-P v2")
@@
 			)
 		)
-		(property "Value" "150"
+		(property "Value" "1k5"
 			(at 144.78 93.98 90)
 			(effects
@@
 			)
 		)
-		(property "Value" "150"
+		(property "Value" "1k5"
 			(at 144.78 116.84 90)
 			(effects
@@
 			)
 		)
-		(property "Value" "150"
+		(property "Value" "1k5"
 			(at 144.78 101.6 90)
 			(effects
@@
 			)
 		)
-		(property "Value" "150"
+		(property "Value" "1k5"
 			(at 144.78 109.22 90)
 			(effects

Commit message: Reworking the KiCAD symbols.
Parts:
- J2: renamed from Header2; symbol 7seg_4d_2x595:pin_header_1-row_2-pin_horizontal -> Drv7Seg2x595:pin_header_1-row_2-pin_horizontal
Changed lines of the file:
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@@
 	)
 	(junction
-		(at 130.81 99.06)
-		(diameter 0)
-		(color 0 0 0 0)
-	)
-	(junction
 		(at 107.95 116.84)
 		(diameter 0)
@@
 	)
 	(symbol
-		(lib_id "7seg_4d_2x595:pin_header_1-row_2-pin_horizontal")
+		(lib_id "Drv7Seg2x595:pin_header_1-row_2-pin_horizontal")
 		(at 196.85 100.33 180)
 		(unit 1)
@@
 		(on_board yes)
 		(dnp no)
-		(property "Reference" "Header2"
+		(property "Reference" "J2"
 			(at 196.85 104.394 0)
 			(effects
@@
 			(project ""
 				(path "/379795a0-c68f-4c94-9399-90603a2bef2e"
-					(reference "Header2")
+					(reference "J2")
 					(unit 1)
 				)

Commit message: Major update of KiCAD files.
Parts:
- D1: renamed from LED1; value LED -> LED1
- DISPLAY1: value 7seg_4d -> display_7seg_4d; symbol 7seg_4d_2x595:7seg_4d -> Drv7Seg2x595:display_7seg_4d
- IC1, IC2: symbol 7seg_4d_2x595:74HC595 -> Drv7Seg2x595:74HC595
- J1: renamed from Header1; value pin_header_1-row_5-pin_horizontal -> INTERFACE; symbol 7seg_4d_2x595:pin_header_1-row_5-pin_horizontal -> Drv7Seg2x595:pin_header_1-row_5-pin_horizontal
- J2: value pin_header_1-row_2-pin_horizontal -> PWR_LED_JMP; footprint Connector_PinHeader_2.54mm:PinHeader_1x02_P2.54mm_Horizontal -> Drv7Seg2x595:PinHeader_1x02_P2.54mm_Horizontal
- Q1, Q2, Q3, Q4: footprint Package_TO_SOT_SMD:SOT-23_Handsoldering -> Package_TO_SOT_SMD:SOT-23
Connections:
- net GND: now also J2.2 (Pin_2); no longer J2.1 (Pin_1)
- net at RLED1.1: now also J2.1 (Pin_1); no longer J2.2 (Pin_2)
Other:
- moved on the sheet: C1, C2
Changed lines of the file:
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@@
 	(wire
 		(pts
-			(xy 191.77 102.87) (xy 191.77 107.95)
-		)
-		(stroke
-			(width 0)
-			(type default)
-		)
-	)
-	(wire
-		(pts
 			(xy 119.38 116.84) (xy 119.38 111.76)
 		)
@@
 	(wire
 		(pts
-			(xy 220.98 95.25) (xy 220.98 90.17)
+			(xy 220.98 96.52) (xy 220.98 90.17)
 		)
 		(stroke
@@
 	(wire
 		(pts
+			(xy 191.77 107.95) (xy 191.77 110.49)
+		)
+		(stroke
+			(width 0)
+			(type default)
+		)
+	)
+	(wire
+		(pts
 			(xy 181.61 72.39) (xy 181.61 64.77)
 		)
@@
 	(wire
 		(pts
-			(xy 220.98 102.87) (xy 220.98 110.49)
+			(xy 220.98 104.14) (xy 220.98 110.49)
 		)
 		(stroke
@@
 	(wire
 		(pts
-			(xy 210.82 102.87) (xy 210.82 110.49)
+			(xy 191.77 105.41) (xy 191.77 102.87)
+		)
+		(stroke
+			(width 0)
+			(type default)
+		)
+	)
+	(wire
+		(pts
+			(xy 210.82 104.14) (xy 210.82 110.49)
 		)
 		(stroke
@@
 	(wire
 		(pts
-			(xy 210.82 90.17) (xy 210.82 95.25)
+			(xy 210.82 90.17) (xy 210.82 96.52)
 		)
 		(stroke
@@
 	)
 	(symbol
-		(lib_name "74HC595_1")
-		(lib_id "7seg_4d_2x595:74HC595")
+		(lib_id "Drv7Seg2x595:74HC595")
 		(at 158.75 69.85 0)
 		(unit 1)
@@
 	(symbol
 		(lib_id "Device:C")
-		(at 220.98 99.06 180)
+		(at 220.98 100.33 180)
 		(unit 1)
 		(exclude_from_sim no)
@@
 		(dnp no)
 		(property "Reference" "C2"
-			(at 225.806 93.726 0)
+			(at 225.806 94.996 0)
 			(effects
 				(font
@@
 		)
 		(property "Value" "0.1 μF"
-			(at 228.092 96.266 0)
+			(at 228.092 97.536 0)
 			(effects
 				(font
@@
 		)
 		(property "Footprint" "Capacitor_SMD:C_0805_2012Metric_Pad1.18x1.45mm_HandSolder"
-			(at 220.0148 95.25 0)
+			(at 220.0148 96.52 0)
 			(effects
 				(font
@@
 		)
 		(property "Datasheet" "~"
-			(at 220.98 99.06 0)
+			(at 220.98 100.33 0)
 			(effects
 				(font
@@
 		)
 		(property "Description" "Unpolarized capacitor"
-			(at 220.98 99.06 0)
+			(at 220.98 100.33 0)
 			(effects
 				(font
@@
 	)
 	(symbol
+		(lib_name "MMBT3904_1")
 		(lib_id "Transistor_BJT:MMBT3904")
 		(at 133.35 93.98 0)
@@
 			)
 		)
-		(property "Footprint" "Package_TO_SOT_SMD:SOT-23_Handsoldering"
+		(property "Footprint" "Package_TO_SOT_SMD:SOT-23"
 			(at 128.27 95.885 0)
 			(effects
@@
 	(symbol
 		(lib_id "Device:C")
-		(at 210.82 99.06 0)
+		(at 210.82 100.33 0)
 		(unit 1)
 		(exclude_from_sim no)
@@
 		(dnp no)
 		(property "Reference" "C1"
-			(at 213.106 93.726 0)
+			(at 213.106 94.996 0)
 			(effects
 				(font
@@
 		)
 		(property "Value" "0.1 μF"
-			(at 211.328 96.266 0)
+			(at 211.328 97.536 0)
 			(effects
 				(font
@@
 		)
 		(property "Footprint" "Capacitor_SMD:C_0805_2012Metric_Pad1.18x1.45mm_HandSolder"
-			(at 211.7852 102.87 0)
+			(at 211.7852 104.14 0)
 			(effects
 				(font
@@
 		)
 		(property "Datasheet" "~"
-			(at 210.82 99.06 0)
+			(at 210.82 100.33 0)
 			(effects
 				(font
@@
 		)
 		(property "Description" "Unpolarized capacitor"
-			(at 210.82 99.06 0)
+			(at 210.82 100.33 0)
 			(effects
 				(font
@@
 		(on_board yes)
 		(dnp no)
-		(fields_autoplaced yes)
-		(property "Reference" "LED1"
+		(property "Reference" "D1"
 			(at 195.58 89.2174 90)
 			(effects
@@
 				)
 				(justify right)
+				(hide yes)
 			)
 		)
-		(property "Value" "LED"
-			(at 195.58 91.7574 90)
+		(property "Value" "LED1"
+			(at 194.31 88.9 90)
 			(effects
 				(font
@@
 				)
 				(justify right)
-				(hide yes)
 			)
 		)
@@
 			)
 		)
+		(property "Sim.Pins" "1=K 2=A"
+			(at 191.77 88.9 0)
+			(effects
+				(font
+					(size 1.27 1.27)
+				)
+				(hide yes)
+			)
+		)
 		(pin "2"
 		)
@@
 			(project ""
 				(path "/379795a0-c68f-4c94-9399-90603a2bef2e"
-					(reference "LED1")
+					(reference "D1")
 					(unit 1)
 				)
@@
 	)
 	(symbol
-		(lib_id "7seg_4d_2x595:7seg_4d")
+		(lib_id "Drv7Seg2x595:display_7seg_4d")
 		(at 113.03 69.85 0)
 		(unit 1)
@@
 			)
 		)
-		(property "Value" "7seg_4d"
+		(property "Value" "display_7seg_4d"
 			(at 113.03 91.186 0)
 			(effects
@@
 			)
 		)
-		(property "Footprint" "Package_TO_SOT_SMD:SOT-23_Handsoldering"
+		(property "Footprint" "Package_TO_SOT_SMD:SOT-23"
 			(at 105.41 113.665 0)
 			(effects
@@
 	)
 	(symbol
-		(lib_id "Drv7Seg2x595:pin_header_1-row_2-pin_horizontal")
-		(at 196.85 100.33 180)
-		(unit 1)
-		(exclude_from_sim no)
-		(in_bom yes)
-		(on_board yes)
-		(dnp no)
-		(property "Reference" "J2"
-			(at 196.85 104.394 0)
-			(effects
-				(font
-					(size 1.27 1.27)
-				)
-			)
-		)
-		(property "Value" "pin_header_1-row_2-pin_horizontal"
-			(at 196.088 104.902 0)
-			(effects
-				(font
-					(size 1.27 1.27)
-				)
-				(hide yes)
-			)
-		)
-		(property "Footprint" "Connector_PinHeader_2.54mm:PinHeader_1x02_P2.54mm_Horizontal"
-			(at 195.072 98.806 0)
-			(effects
-				(font
-					(size 1.27 1.27)
-				)
-				(hide yes)
-			)
-		)
-		(property "Datasheet" "~"
-			(at 196.596 104.14 0)
-			(effects
-				(font
-					(size 1.27 1.27)
-				)
-				(hide yes)
-			)
-		)
-		(property "Description" "Pin header, single row, 2 pins"
-			(at 195.072 101.6 0)
-			(effects
-				(font
-					(size 1.27 1.27)
-				)
-				(hide yes)
-			)
-		)
-		(pin "1"
-		)
-		(pin "2"
-		)
-		(instances
-			(project ""
-				(path "/379795a0-c68f-4c94-9399-90603a2bef2e"
-					(reference "J2")
-					(unit 1)
-				)
-			)
-		)
-	)
-	(symbol
 		(lib_id "Transistor_BJT:MMBT3904")
 		(at 99.06 120.65 0)
@@
 			)
 		)
-		(property "Footprint" "Package_TO_SOT_SMD:SOT-23_Handsoldering"
+		(property "Footprint" "Package_TO_SOT_SMD:SOT-23"
 			(at 93.98 122.555 0)
 			(effects
@@
 	)
 	(symbol
-		(lib_id "7seg_4d_2x595:pin_header_1-row_5-pin_horizontal")
+		(lib_id "Drv7Seg2x595:pin_header_1-row_5-pin_horizontal")
 		(at 196.85 67.31 0)
 		(mirror y)
@@
 		(on_board yes)
 		(dnp no)
-		(property "Reference" "Header1"
+		(property "Reference" "J1"
 			(at 196.85 53.594 0)
 			(effects
@@
 			)
 		)
-		(property "Value" "pin_header_1-row_5-pin_horizontal"
+		(property "Value" "INTERFACE"
 			(at 196.85 74.93 0)
 			(effects
@@
 			(project ""
 				(path "/379795a0-c68f-4c94-9399-90603a2bef2e"
-					(reference "Header1")
+					(reference "J1")
 					(unit 1)
 				)
@@
 	)
 	(symbol
-		(lib_id "7seg_4d_2x595:74HC595")
+		(lib_id "Drv7Seg2x595:74HC595")
 		(at 158.75 106.68 0)
 		(unit 1)
@@
 			)
 		)
-		(property "Footprint" "Package_TO_SOT_SMD:SOT-23_Handsoldering"
+		(property "Footprint" "Package_TO_SOT_SMD:SOT-23"
 			(at 116.84 104.775 0)
 			(effects
@@
 					(unit 1)
 				)
+			)
+		)
+	)
+	(symbol
+		(lib_id "Drv7Seg2x595:pin_header_1-row_2-pin_horizontal")
+		(at 196.85 115.57 0)
+		(mirror y)
+		(unit 1)
+		(exclude_from_sim no)
+		(in_bom yes)
+		(on_board yes)
+		(dnp no)
+		(fields_autoplaced yes)
+		(property "Reference" "J2"
+			(at 196.215 102.87 0)
+			(effects
+				(font
+					(size 1.27 1.27)
+				)
+			)
+		)
+		(property "Value" "PWR_LED_JMP"
+			(at 196.088 110.998 0)
+			(effects
+				(font
+					(size 1.27 1.27)
+				)
+				(hide yes)
+			)
+		)
+		(property "Footprint" "Drv7Seg2x595:PinHeader_1x02_P2.54mm_Horizontal"
+			(at 195.072 117.094 0)
+			(effects
+				(font
+					(size 1.27 1.27)
+				)
+				(hide yes)
+			)
+		)
+		(property "Datasheet" "~"
+			(at 196.596 111.76 0)
+			(effects
+				(font
+					(size 1.27 1.27)
+				)
+				(hide yes)
+			)
+		)
+		(property "Description" "Pin header, single row, 2 pins"
+			(at 195.072 114.3 0)
+			(effects
+				(font
+					(size 1.27 1.27)
+				)
+				(hide yes)
+			)
+		)
+		(pin "2"
+		)
+		(pin "1"
+		)
+		(instances
+			(project ""
+				(path "/379795a0-c68f-4c94-9399-90603a2bef2e"
+					(reference "J2")
+					(unit 1)
+				)
